Commit message: hunter killer mast and droneship

File: mybot_ws/src/droneship/urdf/hunter_killer_mast.urdf (robot description, URDF)
Before this commit: robot hunter_killer_mast, 19 links, 18 joints
Links:
- removed link buax
- removed link hemi1l
- removed link hemi1r
- removed link hemi2l
- removed link hemi2r
- removed link ledport
- removed link ledstarboard
Joints:
- removed joint hemi1l_joint
- removed joint hemi1r_joint
- removed joint hemi2l_joint
- removed joint hemi2r_joint
- removed joint joint_name
- removed joint ledport_joint
- removed joint ledstarboard_joint
- joint communication_module_joint: axis 1 0 0 -> 0 0 0; limit lower=0 upper=1 effort=10 velocity=1 -> (none); type prismatic -> fixed
- joint rod_supporter_joint: limit lower=0 upper=0 effort=0 velocity=0 -> (none)
